Commit message: fix urdf config for navigation

File: interaction_bringup/urdf/interaction_robot.xacro (robot description, xacro)
@@ -7,4 +7,5 @@
   <xacro:include filename="$(find icart_mini_description)/urdf/materials.xacro" />
   <xacro:include filename="$(find orne_description)/urdf/interaction_robot.gazebo"/>
+	<xacro:include filename="$(find icart_mini_description)/urdf/sensors/hokuyo.urdf.xacro"/>
   <!-- <xacro:include filename="$(find icart_mini_description)/urdf/sensors/imu.urdf.xacro"/> <xacro:sensor_imu name="imu" parent="base_link" size="0.05 0.05 0.05">
       <origin xyz="0.04 0.0 0.15" rpy="0 0 3.14"/>
@@ -192,4 +193,8 @@
     </actuator>
   </transmission>
+	<!-- 2d urg -->
+	<xacro:sensor_hokuyo name="hokuyo" parent="base_link">
+		<origin xyz="0.27 0 0.2485" rpy="0 0 0"/>
+	</xacro:sensor_hokuyo>
   <!-- arm -->
   <joint type="fixed" name="arm_base_joint">

Commit message: add kinect to urdf and ar_tag launch in elevator_recognition

File: interaction_bringup/urdf/interaction_robot.xacro (robot description, xacro)
@@ -197,4 +197,19 @@
 		<origin xyz="0.27 0 0.2485" rpy="0 0 0"/>
 	</xacro:sensor_hokuyo>
+	<!-- kinect -->
+  <joint type="fixed" name="kinect_joint">
+    <parent link="base_link"/>
+    <child link="camera_link"/>
+    <origin xyz="0.14 0.0 1.40" rpy="0 0.5 0"/>
+  </joint>
+   <link name="camera_link">
+    <visual name="visual">
+      <origin xyz="0.0 0 0.0" rpy="0 0.5 0"/>
+      <geometry>
+	      <box size=".05 .2 .05"/>
+      </geometry>
+      <material name="orange"/>
+    </visual>
+  </link>
   <!-- arm -->
   <joint type="fixed" name="arm_base_joint">

Commit message: fix 2d lidar pos in urdf

File: interaction_bringup/urdf/interaction_robot.xacro (robot description, xacro)
@@ -195,5 +195,5 @@
 	<!-- 2d urg -->
 	<xacro:sensor_hokuyo name="hokuyo" parent="base_link">
-		<origin xyz="0.27 0 0.2485" rpy="0 0 0"/>
+		<origin xyz="0.29 0 0.2485" rpy="0 0 0"/>
 	</xacro:sensor_hokuyo>
 	<!-- kinect -->
@@ -213,4 +213,18 @@
   </link>
   <!-- arm -->
+  <joint type="fixed" name="up_bottun_finter">
+    <parent link="base_link"/>
+    <child link="up_bottun_bar"/>
+    <origin xyz="0.53 0.0 1.22" rpy="0 0 0"/>
+  </joint>
+  <link name="up_bottun_bar">
+    <visual name="visual">
+      <origin xyz="-0.25 0 0.0" rpy="0 0 0"/>
+      <geometry>
+	      <box size=".50 .02 .02"/>
+      </geometry>
+      <material name="orange"/>
+    </visual>
+  </link>
   <joint type="fixed" name="arm_base_joint">
     <parent link="base_link"/>

Commit message: update

File: interaction_bringup/urdf/interaction_robot.xacro (robot description, xacro)
@@ -201,5 +201,5 @@
     <parent link="base_link"/>
     <child link="camera_link"/>
-    <origin xyz="0.14 0.0 1.40" rpy="0 0.5 0"/>
+    <origin xyz="0.20 0.05 1.40" rpy="0 0.43 0.04"/>
   </joint>
    <link name="camera_link">
@@ -213,17 +213,10 @@
   </link>
   <!-- arm -->
-  <joint type="fixed" name="up_bottun_finter">
+  <joint type="fixed" name="up_bottun_bar_joint">
     <parent link="base_link"/>
     <child link="up_bottun_bar"/>
-    <origin xyz="0.53 0.0 1.22" rpy="0 0 0"/>
+    <origin xyz="0.82 0.0 1.3" rpy="0 0 0"/>
   </joint>
   <link name="up_bottun_bar">
-    <visual name="visual">
-      <origin xyz="-0.25 0 0.0" rpy="0 0 0"/>
-      <geometry>
-	      <box size=".50 .02 .02"/>
-      </geometry>
-      <material name="orange"/>
-    </visual>
   </link>
   <joint type="fixed" name="arm_base_joint">

Commit message: add joint 4 limit

File: interaction_bringup/urdf/interaction_robot.xacro (robot description, xacro)
@@ -310,5 +310,5 @@
     <origin xyz="-0.05 0.0 0.23" rpy="0 0 3.14"/>
     <axis xyz="0 1 0" rpy="0 0 0"/>
-    <limit effort="100" velocity="100.0"  lower="-1.57" upper="1.57" />
+    <limit effort="100" velocity="100.0"  lower="0.0" upper="1.57" />
   </joint>
   <link name="arm_link_5">

Commit message: update

File: interaction_bringup/urdf/interaction_robot.xacro (robot description, xacro)
@@ -198,5 +198,5 @@
 	</xacro:sensor_hokuyo>
 	<!-- kinect -->
-  <joint type="fixed" name="kinect_joint">
+  <joint type="fixed" name="neck_joint_0">
     <parent link="base_link"/>
     <child link="camera_link"/>
